Commit message: demo version

File: src/f450_drone_description/urdf/f450.urdf.xacro (robot description, xacro)
@@ -39,6 +39,6 @@
     <visual>
       <origin xyz="0 0 0" rpy="0 0 0"/>
-      <geometry><box size="0.10 0.10 0.07"/></geometry>
-      <material name="dark_gray"><color rgba="0.1 0.1 0.1 0.9"/></material>
+      <geometry><box size="0.10 0.10 0.05"/></geometry>
+      <material name="dark_gray"><color rgba="0.25 0.25 0.25 0.98"/></material>
     </visual>
     <collision>
@@ -49,22 +49,22 @@
   </link>
 <!-- Arms + motor + rotors (x4) -->
-  <xacro:macro name="arm_with_rotor" params="name angle color_name color_rgba">
-<!-- arm link -->
-<link name="${name}_arm">
-  <visual>
-    <origin xyz="${frame_radius/4} 0 0" rpy="0 0 0"/>  <!-- Offset = half of arm length -->
-    <geometry><box size="${frame_radius/2} 0.02 0.02"/></geometry>  <!-- 25cm long -->
-    <material name="${color_name}"><color rgba="${color_rgba}"/></material>
-  </visual>
-  <collision>
-    <origin xyz="${frame_radius/4} 0 0" rpy="0 0 0"/>
-    <geometry><box size="${frame_radius/2} 0.02 0.02"/></geometry>
-  </collision>
-  <inertial>
-    <origin xyz="${frame_radius/4} 0 0" rpy="0 0 0"/>
-    <mass value="${arm_mass}"/>
-    <inertia ixx="0.0005" iyy="0.002" izz="0.002" ixy="0" ixz="0" iyz="0"/>
-  </inertial>
-</link>
+<xacro:macro name="arm_with_rotor" params="name angle color_name color_rgba">
+    <!-- arm link -->
+    <link name="${name}_arm">
+      <visual>
+        <origin xyz="${frame_radius/4} 0 0" rpy="0 0 0"/>  <!-- Offset = half of arm length -->
+        <geometry><box size="${frame_radius/2} 0.02 0.02"/></geometry>  <!-- 25cm long -->
+        <material name="${color_name}"><color rgba="${color_rgba}"/></material>
+      </visual>
+      <collision>
+        <origin xyz="${frame_radius/4} 0 0" rpy="0 0 0"/>
+        <geometry><box size="${frame_radius/2} 0.02 0.02"/></geometry>
+      </collision>
+      <inertial>
+        <origin xyz="${frame_radius/4} 0 0" rpy="0 0 0"/>
+        <mass value="${arm_mass}"/>
+        <inertia ixx="0.0005" iyy="0.002" izz="0.002" ixy="0" ixz="0" iyz="0"/>
+      </inertial>
+    </link>
     <joint name="base_to_${name}_arm" type="fixed">
       <origin xyz="0 0 0" rpy="0 0 ${angle}"/>
@@ -75,10 +75,10 @@
     <link name="${name}_motor">
       <visual>
-        <origin xyz="${frame_radius/2.0} 0 0.0" rpy="0 0 0"/>
-        <geometry><cylinder radius="0.015" length="0.035"/></geometry>
+        <origin xyz="${frame_radius/2.0-0.011} 0 0.0175" rpy="0 0 0"/>
+        <geometry><cylinder radius="0.010" length="0.035"/></geometry>
         <material name="red"><color rgba="1.0 0.0 0.0 1.0"/></material>
       </visual>
       <collision>
-        <origin xyz="${frame_radius/2.0} 0 0.0" rpy="0 0 0"/>
+        <origin xyz="${frame_radius/2.0-0.011} 0 0.0175" rpy="0 0 0"/>
         <geometry><cylinder radius="0.015" length="0.035"/></geometry>
       </collision>
@@ -92,10 +92,10 @@
     <link name="${name}_blade">
       <visual>
-        <origin xyz="${frame_radius/2.0} 0 0.045" rpy="0 0 0"/>
+        <origin xyz="${frame_radius/2.0-0.011} 0 0.045" rpy="0 0 0"/>
         <geometry><cylinder radius="0.11" length="0.005"/></geometry>
         <material name="grey"><color rgba="0.6 0.6 0.6 0.2"/></material>
       </visual>
       <collision>
-        <origin xyz="${frame_radius/2.0} 0 0.045" rpy="0 0 0"/>
+        <origin xyz="${frame_radius/2.0-0.011} 0 0.045" rpy="0 0 0"/>
         <geometry><cylinder radius="0.11" length="0.005"/></geometry>
       </collision>
